File: 01_USB_Charging.kicad_sch (KiCad schematic)
At the start: 22 parts, among them J1 USB4105-GF-A, J2 Conn_01x03_Pin, U4 ETA6003Q3Q

Commit message: removed firmware
Parts:
- C1, C2: Design_note 1nF / 10V -> (none); Voltage 10V X7R -> (none)
- C3: Design_note 1uF / 10V -> (none); Voltage 10V X7R -> (none)
- C4: Design_note 100nF / 10V -> (none); Voltage 10V X7R -> (none)
- R1, R4: value 5.1k 1% -> 5.1k
- R2, R3, R5, R6: value 100k 1% -> 100k
Connections:
- net CC1 is gone; now on an unnamed net: R2.2
- net CC2 is gone; now on an unnamed net: R5.1
- net GND: now also R1.1, R4.1; no longer R1.2, R4.2
- net at J1.B5 (CC2): now also R1.2; no longer R1.1
- net at J1.A5 (CC1): now also R4.2; no longer R4.1
Other:
- note removed: "External protected 1S pack required. J4: bonded 100k NTC; confirm thermistor curve and thresholds."
- note removed: "IP2312 fixed 4.20V variant only; 135k sets nominal 1A. Confirm selected cell permits 1C charge."
- note removed: "L2 changed to 1uH per charger reference; select >=4A saturation part and verify temperature."
- note removed: "No system power path: charge only with playback stopped; verify termination with MCU load."
- note removed: "Q3 default OFF. Enable charging only after valid USB-C >=1.5A advertisement; never assume 2A."
- moved on the sheet: C1, C2, C3, C4, D1, R1, R2, R3, R4, R5, R6

Commit message: ??
Parts:
- R2, R5: value 100k -> 510k
Other:
- note removed: "REVIEW DRAFT | Labels are electrical connections across all sheets"
Changed lines of the file:
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@@
 		(comment 1 "NOT FOR FABRICATION - see DESIGN_NOTES.md")
 	)
-	(text "REVIEW DRAFT  |  Labels are electrical connections across all sheets"
-		(exclude_from_sim no)
-		(at 248.92 87.376 0)
-		(effects
-			(font
-				(size 1.27 1.27)
-			)
-			(justify left top)
-		)
-	)
 	(text "01 USB CHARGING"
 		(exclude_from_sim no)
@@
 			)
 		)
-		(property "Value" "100k"
+		(property "Value" "510k"
 			(at 203.2 114.554 90)
 			(show_name no)
@@
 			)
 		)
-		(property "Value" "100k"
+		(property "Value" "510k"
 			(at 203.2 119.634 90)
 			(show_name no)
