File: 02_Power.kicad_sch (KiCad schematic)
At the start: 15 parts, among them U6 TLV62568DBVR, U7 RT9080

Commit message: removed firmware
Parts:
- L1: value 2.2uH DFE201210U-1R0M=P2 -> DFE201210U-1R0M
- R13: value 200k 1% -> 200k
- R14, R21: value 100k 1% -> 100k
- R20: value 330k 1% -> 330k
Changed lines of the file:
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@@
 			)
 		)
-		(property "Value" "330k 1%"
+		(property "Value" "330k"
 			(at 233.934 174.244 90)
 			(show_name no)
@@
 			)
 		)
-		(property "Value" "100k 1%"
+		(property "Value" "100k"
 			(at 236.41 185.42 0)
 			(show_name no)
@@
 			)
 		)
-		(property "Value" "100k 1%"
+		(property "Value" "100k"
 			(at 338.074 198.374 0)
 			(show_name no)
@@
 			)
 		)
-		(property "Value" "200k 1%"
+		(property "Value" "200k"
 			(at 349.758 194.246 90)
 			(show_name no)
@@
 			)
 		)
-		(property "Value" "2.2uH DFE201210U-1R0M=P2"
+		(property "Value" "DFE201210U-1R0M"
 			(at 357.124 185.928 90)
 			(show_name no)

Commit message: ??
Parts:
- added R11: 100k, Resistor_SMD:R_0402_1005Metric, symbol Device:R
- added R17: 510k, Resistor_SMD:R_0402_1005Metric, symbol Device:R
Connections:
- net GND: now also R11.2
- net VBAT: now also R17.1
- new net VBAT_ADC: R11.1, R17.2
Other:
- note removed: "REVIEW DRAFT | Labels are electrical connections across all sheets"
