File: 03_MCU_RF.kicad_sch (KiCad schematic)
At the start: 42 parts, among them J5 TC2050, U1 nRF5340-QKAA, U5 SC7A20, Y1 32MHz / CL=8pF / 10ppm

Commit message: removed firmware
Parts:
- C23, C24, C25: Voltage 10V X7R -> (none)
- C26, C29, C30, C31, C32, C33, C34, C35, C36: Design_note 100nF / 10V -> (none); Voltage 10V X7R -> (none)
- C27: Design_note 1uF / 10V -> (none); Voltage 10V X7R -> (none)
- C28: Design_note 4.7uF / 10V -> (none); Voltage 10V X7R -> (none)
- C37, C40: footprint Capacitor_SMD:C_0603_1608Metric -> Capacitor_SMD:C_0402_1005Metric; Design_note 4.7uF / 10V -> (none); Voltage 10V X7R -> (none)
- R10: value R -> 0R
- R22: Design_note 0R / antenna tuning -> (none)
- R23: Design_note 10k -> (none)
- R25, R26, R27, R28: Design_note 4.7k -> (none)
- R29, R30, R31, R32: Design_note 22R -> (none)
Connections:
- net USB_DET: now reaches U1.A17 (P1.13)
- net VBAT_ADC renamed VBAT
- no-connect marks 37 -> 36
Changed lines of the file:
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@@
 	)
 	(no_connect
-		(at 326.39 271.78)
-	)
-	(no_connect
 		(at 326.39 198.12)
 	)
@@
 	(wire
 		(pts
+			(xy 326.39 271.78) (xy 330.2 271.78)
+		)
+		(stroke
+			(width 0)
+			(type default)
+		)
+	)
+	(wire
+		(pts
 			(xy 83.82 157.48) (xy 83.82 156.21)
 		)
@@
 	(wire
 		(pts
-			(xy 326.39 226.06) (xy 328.93 226.06)
+			(xy 326.39 226.06) (xy 330.2 226.06)
 		)
 		(stroke
@@
 	)
 	(label "ACC_INT2"
-		(at 328.93 226.06 0)
+		(at 330.2 226.06 0)
 		(effects
 			(font
@@
 		)
 	)
+	(global_label "USB_DET"
+		(shape passive)
+		(at 330.2 271.78 0)
+		(fields_autoplaced yes)
+		(effects
+			(font
+				(size 1.27 1.27)
+			)
+			(justify left)
+		)
+		(property "Intersheetrefs" "${INTERSHEET_REFS}"
+			(at 339.3121 271.78 0)
+			(hide yes)
+			(show_name no)
+			(do_not_autoplace no)
+			(effects
+				(font
+					(size 1.27 1.27)
+				)
+				(justify left)
+			)
+		)
+	)
 	(global_label "VDD_1V8"
 		(shape bidirectional)
@@
 		)
 	)
-	(global_label "I2S_DATA"
+	(global_label "VBAT"
 		(shape bidirectional)
-		(at 356.87 238.76 0)
+		(at 331.47 170.18 0)
 		(effects
 			(font
@@
 		)
 		(property "Intersheetrefs" "${INTERSHEET_REFS}"
-			(at 356.87 238.76 0)
+			(at 331.47 170.18 0)
 			(hide yes)
 			(show_name no)
@@
 		)
 	)
-	(global_label "D_N"
+	(global_label "I2S_DATA"
 		(shape bidirectional)
-		(at 331.47 284.48 0)
+		(at 356.87 238.76 0)
 		(effects
 			(font
@@
 		)
 		(property "Intersheetrefs" "${INTERSHEET_REFS}"
-			(at 331.47 284.48 0)
+			(at 356.87 238.76 0)
 			(hide yes)
 			(show_name no)
@@
 		)
 	)
-	(global_label "VBAT_ADC"
+	(global_label "D_N"
 		(shape bidirectional)
-		(at 331.47 170.18 0)
+		(at 331.47 284.48 0)
 		(effects
 			(font
@@
 		)
 		(property "Intersheetrefs" "${INTERSHEET_REFS}"
-			(at 331.47 170.18 0)
+			(at 331.47 284.48 0)
 			(hide yes)
 			(show_name no)
@@
 			)
 		)
-		(property "Voltage" "10V X7R"
+		(property "Voltage" ""
 			(at 303.72 118.11 0)
 			(show_name no)
@@
 			)
 		)
-		(property "Design_note" "100nF / 10V"
+		(property "Design_note" ""
 			(at 299.72 114.3 0)
 			(hide yes)
@@
 			)
 		)
-		(property "Voltage" "10V X7R"
+		(property "Voltage" ""
 			(at 354.52 118.11 0)
 			(show_name no)
@@
 			)
 		)
-		(property "Design_note" "100nF / 10V"
+		(property "Design_note" ""
 			(at 350.52 114.3 0)
 			(hide yes)
@@
 			)
 		)
-		(property "Voltage" "10V X7R"
+		(property "Voltage" ""
 			(at 338.01 118.11 0)
 			(show_name no)
@@
 			)
 		)
-		(property "Design_note" "100nF / 10V"
+		(property "Design_note" ""
 			(at 334.01 114.3 0)
 			(hide yes)
@@
 			)
 		)
-		(property "Value" "R"
+		(property "Value" "0R"
 			(at 205.74 260.35 90)
 			(show_name no)
@@
 			)
 		)
-		(property "Design_note" "22R"
+		(property "Design_note" ""
 			(at 350.52 218.44 0)
 			(hide yes)
@@
 			)
 		)
-		(property "Voltage" "10V X7R"
+		(property "Voltage" ""
 			(at 320.23 118.11 0)
 			(show_name no)
@@
 			)
 		)
-		(property "Design_note" "100nF / 10V"
+		(property "Design_note" ""
 			(at 316.23 114.3 0)
 			(hide yes)
@@
 			)
 		)
-		(property "Design_note" "22R"
+		(property "Design_note" ""
 			(at 350.52 238.76 0)
 			(hide yes)
@@
 			)
 		)
-		(property "Voltage" "10V X7R"
+		(property "Voltage" ""
 			(at 241.49 118.11 0)
 			(show_name no)
@@
 			)
 		)
-		(property "Design_note" "100nF / 10V"
+		(property "Design_note" ""
 			(at 237.49 114.3 0)
 			(hide yes)
@@
 			)
 		)
-		(property "Voltage" "10V X7R"
+		(property "Voltage" ""
 			(at 287.21 118.11 0)
 			(show_name no)
@@
 			)
 		)
-		(property "Design_note" "100nF / 10V"
+		(property "Design_note" ""
 			(at 283.21 114.3 0)
 			(hide yes)
@@
 			)
 		)
-		(property "Voltage" "10V X7R"
+		(property "Voltage" ""
 			(at 271.97 118.11 0)
 			(show_name no)
@@
 			)
 		)
-		(property "Design_note" "100nF / 10V"
+		(property "Design_note" ""
 			(at 267.97 114.3 0)
 			(hide yes)
@@
 			)
 		)
-		(property "Design_note" "4.7k"
+		(property "Design_note" ""
 			(at 350.52 195.58 0)
 			(hide yes)
@@
 			)
 		)
-		(property "Design_note" "4.7k"
+		(property "Design_note" ""
 			(at 337.82 248.92 0)
 			(hide yes)
@@
 			)
 		)
-		(property "Design_note" "0R / antenna tuning"
+		(property "Design_note" ""
 			(at 228.6 264.16 0)
 			(hide yes)
@@
 			)
 		)
-		(property "Design_note" "22R"
+		(property "Design_note" ""
 			(at 350.52 213.36 0)
 			(hide yes)
@@
 			)
 		)
-		(property "Footprint" "Capacitor_SMD:C_0603_1608Metric"
+		(property "Footprint" "Capacitor_SMD:C_0402_1005Metric"
 			(at 367.03 114.3 0)
 			(hide yes)
@@
 			)
 		)
-		(property "Voltage" "10V X7R"
+		(property "Voltage" ""
 			(at 371.03 118.11 0)
 			(show_name no)
@@
 			)
 		)
-		(property "Design_note" "4.7uF / 10V"
+		(property "Design_note" ""
 			(at 367.03 114.3 0)
 			(hide yes)
@@
 			)
 		)
-		(property "Voltage" "10V X7R"
+		(property "Voltage" ""
 			(at 251.65 255.27 0)
 			(show_name no)
@@
 			)
 		)
-		(property "Design_note" "10k"
+		(property "Design_note" ""
 			(at 238.76 153.67 0)
 			(hide yes)
@@
 			)
 		)
-		(property "Design_note" "4.7k"
+		(property "Design_note" ""
 			(at 350.52 187.96 0)
 			(hide yes)
@@
 			)
 		)
-		(property "Voltage" "10V X7R"
+		(property "Voltage" ""
 			(at 245.3 295.91 0)
 			(show_name no)
@@
 			)
 		)
-		(property "Design_note" "100nF / 10V"
+		(property "Design_note" ""
 			(at 241.3 292.1 0)
 			(hide yes)
@@
 			)
 		)
-		(property "Voltage" "10V X7R"
+		(property "Voltage" ""
 			(at 259.27 295.91 0)
+			(hide yes)
 			(show_name no)
 			(do_not_autoplace no)
@@
 			)
 		)
-		(property "Design_note" "1uF / 10V"
+		(property "Design_note" ""
 			(at 255.27 292.1 0)
 			(hide yes)
@@
 			)
 		)
-		(property "Design_note" "22R"
+		(property "Design_note" ""
 			(at 350.52 223.52 0)
 			(hide yes)
@@
 			)
 		)
-		(property "Design_note" "4.7k"
+		(property "Design_note" ""
 			(at 345.44 248.92 0)
 			(hide yes)
@@
 			)
 		)
-		(property "Voltage" "10V X7R"
+		(property "Voltage" ""
 			(at 231.33 295.91 0)
 			(show_name no)
@@
 			)
 		)
-		(property "Design_note" "4.7uF / 10V"
+		(property "Design_note" ""
 			(at 227.33 292.1 0)
 			(hide yes)
@@
 			)
 		)
-		(property "Voltage" "10V X7R"
+		(property "Voltage" ""
 			(at 251.65 227.33 0)
 			(show_name no)
@@
 			)
 		)
-		(property "Voltage" "10V X7R"
+		(property "Voltage" ""
 			(at 256.73 118.11 0)
 			(show_name no)
@@
 			)
 		)
-		(property "Design_note" "100nF / 10V"
+		(property "Design_note" ""
 			(at 252.73 114.3 0)
 			(hide yes)
@@
 			)
 		)
-		(property "Voltage" "10V X7R"
+		(property "Voltage" ""
 			(at 238.95 227.33 0)
 			(show_name no)
@@
 			)
 		)
-		(property "Footprint" "Capacitor_SMD:C_0603_1608Metric"
+		(property "Footprint" "Capacitor_SMD:C_0402_1005Metric"
 			(at 383.54 114.3 0)
 			(hide yes)
@@
 			)
 		)
-		(property "Voltage" "10V X7R"
+		(property "Voltage" ""
 			(at 387.54 118.11 0)
 			(show_name no)
@@
 			)
 		)
-		(property "Design_note" "4.7uF / 10V"
+		(property "Design_note" ""
 			(at 383.54 114.3 0)
 			(hide yes)

Commit message: ??
Parts:
- R25, R26, R27, R28: value 4.7k -> 10k
Connections:
- net VBAT is gone; now on net VBAT_ADC: U1.AB2 (AIN2/P0.06)
- net CC2_ADC: now also U1.W1 (NFC1/P0.02)
- net VDD_1V8: now also R24.2, R25.2, R26.2, R27.2, R28.2
- net VDD_nRF: no longer R24.2, R25.2, R26.2, R27.2, R28.2
- net VBAT_ADC: now reaches U1.AA1 (NFC2/P0.03)
- no-connect marks 36 -> 34
Other:
- note removed: "REVIEW DRAFT | Labels are electrical connections across all sheets"
Changed lines of the file:
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@@
 		)
 	)
-	(text "REVIEW DRAFT  |  Labels are electrical connections across all sheets"
-		(exclude_from_sim no)
-		(at 19.304 27.432 0)
-		(effects
-			(font
-				(size 1.27 1.27)
-			)
-			(justify left top)
-		)
-	)
 	(text "Unused GPIO / unused interfaces explicitly NC; use calibrated LFRC."
 		(exclude_from_sim no)
@@
 	(text "03 MCU RF"
 		(exclude_from_sim no)
-		(at 19.304 19.432 0)
+		(at 267.716 82.678 0)
 		(effects
 			(font
@@
 	)
 	(junction
+		(at 345.44 167.64)
+		(diameter 0)
+		(color 0 0 0 0)
+	)
+	(junction
 		(at 210.82 264.16)
 		(diameter 0)
@@
 	)
 	(no_connect
-		(at 326.39 160.02)
-	)
-	(no_connect
 		(at 77.47 172.72)
 	)
@@
 	)
 	(no_connect
-		(at 326.39 162.56)
-	)
-	(no_connect
 		(at 326.39 198.12)
 	)
@@
 	(wire
 		(pts
-			(xy 326.39 167.64) (xy 331.47 167.64)
+			(xy 326.39 167.64) (xy 345.44 167.64)
 		)
 		(stroke
@@
 	(wire
 		(pts
+			(xy 326.39 162.56) (xy 331.47 162.56)
+		)
+		(stroke
+			(width 0)
+			(type default)
+		)
+	)
+	(wire
+		(pts
 			(xy 247.65 218.44) (xy 247.65 219.71)
 		)
@@
 	(wire
 		(pts
+			(xy 345.44 167.64) (xy 351.79 167.64)
+		)
+		(stroke
+			(width 0)
+			(type default)
+		)
+	)
+	(wire
+		(pts
 			(xy 260.35 157.48) (xy 255.27 157.48)
 		)
@@
 	(wire
 		(pts
+			(xy 345.44 160.02) (xy 326.39 160.02)
+		)
+		(stroke
+			(width 0)
+			(type default)
+		)
+	)
+	(wire
+		(pts
 			(xy 157.48 154.94) (xy 160.02 154.94)
 		)
@@
 	(wire
 		(pts
+			(xy 345.44 167.64) (xy 345.44 160.02)
+		)
+		(stroke
+			(width 0)
+			(type default)
+		)
+	)
+	(wire
+		(pts
 			(xy 223.52 273.05) (xy 223.52 274.32)
 		)
@@
 		)
 	)
+	(global_label "VDD_1V8"
+		(shape bidirectional)
+		(at 356.87 195.58 0)
+		(effects
+			(font
+				(size 1 1)
+			)
+			(justify left)
+		)
+		(property "Intersheetrefs" "${INTERSHEET_REFS}"
+			(at 356.87 195.58 0)
+			(hide yes)
+			(show_name no)
+			(do_not_autoplace no)
+			(effects
+				(font
+					(size 1 1)
+				)
+			)
+		)
+	)
 	(global_label "VDD_nRF"
 		(shape passive)
@@
 		)
 	)
+	(global_label "VBAT_ADC"
+		(shape bidirectional)
+		(at 331.47 162.56 0)
+		(effects
+			(font
+				(size 1 1)
+			)
+			(justify left)
+		)
+		(property "Intersheetrefs" "${INTERSHEET_REFS}"
+			(at 331.47 162.56 0)
+			(hide yes)
+			(show_name no)
+			(do_not_autoplace no)
+			(effects
+				(font
+					(size 1 1)
+				)
+			)
+		)
+	)
 	(global_label "I2C_SDA"
 		(shape bidirectional)
@@
 		)
 	)
-	(global_label "VDD_nRF"
-		(shape passive)
-		(at 290.83 142.24 90)
-		(fields_autoplaced yes)
+	(global_label "VDD_1V8"
+		(shape bidirectional)
+		(at 356.87 242.57 0)
 		(effects
 			(font
-				(size 1.27 1.27)
+				(size 1 1)
 			)
 			(justify left)
 		)
 		(property "Intersheetrefs" "${INTERSHEET_REFS}"
-			(at 290.83 133.1279 90)
+			(at 356.87 242.57 0)
 			(hide yes)
 			(show_name no)
@@
 			(effects
 				(font
-					(size 1.27 1.27)
+					(size 1 1)
 				)
-				(justify left)
 			)
 		)
@@
 	(global_label "VDD_nRF"
 		(shape passive)
-		(at 356.87 177.8 0)
+		(at 290.83 142.24 90)
 		(fields_autoplaced yes)
 		(effects
@@
 		)
 		(property "Intersheetrefs" "${INTERSHEET_REFS}"
-			(at 365.9821 177.8 0)
+			(at 290.83 133.1279 90)
 			(hide yes)
 			(show_name no)
@@
 		)
 	)
-	(global_label "VBAT"
+	(global_label "VBAT_ADC"
 		(shape bidirectional)
 		(at 331.47 170.18 0)
@@
 		)
 	)
-	(global_label "VDD_nRF"
-		(shape passive)
+	(global_label "VDD_1V8"
+		(shape bidirectional)
 		(at 356.87 187.96 0)
-		(fields_autoplaced yes)
 		(effects
 			(font
-				(size 1.27 1.27)
+				(size 1 1)
 			)
 			(justify left)
 		)
 		(property "Intersheetrefs" "${INTERSHEET_REFS}"
-			(at 365.9821 187.96 0)
+			(at 356.87 187.96 0)
 			(hide yes)
 			(show_name no)
@@
 			(effects
 				(font
-					(size 1.27 1.27)
+					(size 1 1)
 				)
-				(justify left)
 			)
 		)
@@
 		)
 	)
-	(global_label "VDD_nRF"
-		(shape passive)
-		(at 356.87 242.57 0)
-		(fields_autoplaced yes)
-		(effects
-			(font
-				(size 1.27 1.27)
-			)
-			(justify left)
-		)
-		(property "Intersheetrefs" "${INTERSHEET_REFS}"
-			(at 365.9821 242.57 0)
-			(hide yes)
-			(show_name no)
-			(do_not_autoplace no)
-			(effects
-				(font
-					(size 1.27 1.27)
-				)
-				(justify left)
-			)
-		)
-	)
-	(global_label "VDD_nRF"
-		(shape passive)
-		(at 356.87 195.58 0)
-		(fields_autoplaced yes)
-		(effects
-			(font
-				(size 1.27 1.27)
-			)
-			(justify left)
-		)
-		(property "Intersheetrefs" "${INTERSHEET_REFS}"
-			(at 365.9821 195.58 0)
-			(hide yes)
-			(show_name no)
-			(do_not_autoplace no)
-			(effects
-				(font
-					(size 1.27 1.27)
-				)
-				(justify left)
-			)
-		)
-	)
 	(global_label "MCU_RESET"
 		(shape bidirectional)
@@
 	(global_label "CC2_ADC"
 		(shape bidirectional)
-		(at 331.47 167.64 0)
+		(at 351.79 167.64 0)
 		(effects
 			(font
@@
 		)
 		(property "Intersheetrefs" "${INTERSHEET_REFS}"
-			(at 331.47 167.64 0)
+			(at 351.79 167.64 0)
 			(hide yes)
 			(show_name no)
@@
 					(size 1 1)
 				)
+				(justify right)
 			)
 		)
@@
 		)
 	)
+	(global_label "VDD_1V8"
+		(shape bidirectional)
+		(at 356.87 177.8 0)
+		(effects
+			(font
+				(size 1 1)
+			)
+			(justify left)
+		)
+		(property "Intersheetrefs" "${INTERSHEET_REFS}"
+			(at 356.87 177.8 0)
+			(hide yes)
+			(show_name no)
+			(do_not_autoplace no)
+			(effects
+				(font
+					(size 1 1)
+				)
+			)
+		)
+	)
 	(global_label "VDD_nRF"
 		(shape passive)
@@
 			)
 		)
-		(property "Value" "4.7k"
+		(property "Value" "10k"
 			(at 354.584 193.548 90)
 			(show_name no)
@@
 			)
 		)
-		(property "Value" "4.7k"
+		(property "Value" "10k"
 			(at 336.296 250.444 0)
 			(show_name no)
@@
 			)
 		)
-		(property "Value" "4.7k"
+		(property "Value" "10k"
 			(at 354.584 185.928 90)
 			(show_name no)
@@
 			)
 		)
-		(property "Value" "4.7k"
+		(property "Value" "10k"
 			(at 343.916 249.936 0)
 			(show_name no)
