File: 04_DAC_Left.kicad_sch (KiCad schematic)
At the start: 18 parts, among them U2 CS43131-CNZR / L mono

Commit message: removed firmware
Parts:
- R36: value 2R 1% -> 2R
Changed lines of the file:
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@@
 			)
 		)
-		(property "Value" "2R 1%"
+		(property "Value" "2R"
 			(at 122.11 106.68 0)
 			(show_name no)

Commit message: ??
Other:
- note removed: "REVIEW DRAFT | Labels are electrical connections across all sheets"
Changed lines of the file:
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@@
-		)
-	)
-	(text "REVIEW DRAFT  |  Labels are electrical connections across all sheets"
-		(exclude_from_sim no)
-		(at 177.8 45.846 0)
-		(effects
-			(font
-				(size 1.27 1.27)
-			)
-			(justify left top)
 		)
 	)
@@
 	(text "04 DAC"
 		(exclude_from_sim no)
-		(at 177.8 37.846 0)
+		(at 177.038 49.022 0)
 		(effects
 			(font
