File: 06_Balanced_Output.kicad_sch (KiCad schematic)
At the start: 4 parts

Commit message: removed firmware
Parts:
- TP1, TP2, TP3, TP4: footprint Connector_Wire:SolderWirePad_1x01_SMD_1.5x3mm -> Connector_PinHeader_2.00mm:PinHeader_1x01_P2.00mm_Vertical; now not fitted
Changed lines of the file:
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@@
 		(on_board yes)
 		(in_pos_files yes)
-		(dnp no)
+		(dnp yes)
 		(property "Reference" "TP4"
 			(at 261.112 119.38 90)
@@
 			)
 		)
-		(property "Footprint" "Connector_Wire:SolderWirePad_1x01_SMD_1.5x3mm"
+		(property "Footprint" "Connector_PinHeader_2.00mm:PinHeader_1x01_P2.00mm_Vertical"
 			(at 254 119.38 0)
 			(hide yes)
@@
 		(on_board yes)
 		(in_pos_files yes)
-		(dnp no)
+		(dnp yes)
 		(property "Reference" "TP3"
 			(at 261.112 114.3 90)
@@
 			)
 		)
-		(property "Footprint" "Connector_Wire:SolderWirePad_1x01_SMD_1.5x3mm"
+		(property "Footprint" "Connector_PinHeader_2.00mm:PinHeader_1x01_P2.00mm_Vertical"
 			(at 254 114.3 0)
 			(hide yes)
@@
 		(on_board yes)
 		(in_pos_files yes)
-		(dnp no)
+		(dnp yes)
 		(property "Reference" "TP2"
 			(at 261.112 108.966 90)
@@
 			)
 		)
-		(property "Footprint" "Connector_Wire:SolderWirePad_1x01_SMD_1.5x3mm"
+		(property "Footprint" "Connector_PinHeader_2.00mm:PinHeader_1x01_P2.00mm_Vertical"
 			(at 254 109.22 0)
 			(hide yes)
@@
 		(on_board yes)
 		(in_pos_files yes)
-		(dnp no)
+		(dnp yes)
 		(property "Reference" "TP1"
 			(at 261.112 104.14 90)
@@
 			)
 		)
-		(property "Footprint" "Connector_Wire:SolderWirePad_1x01_SMD_1.5x3mm"
+		(property "Footprint" "Connector_PinHeader_2.00mm:PinHeader_1x01_P2.00mm_Vertical"
 			(at 254 104.14 0)
 			(hide yes)

Commit message: ??
Other:
- note removed: "Configuration links and JP9 must agree before power-up; this design does not hot-switch modes."
- note removed: "ECO / HD800: bridge each 3-pad selector 1-2; leave all four TURBO INPUT links open; JP9=1-2."
- note removed: "Eco may omit U5/U8, U4, Q1/Q2 and amplifier support parts entirely. Turbo populates them."
- note removed: "L-/R- are driven outputs. OPA1688 current does not establish the original 250mW/18ohm target."
- note removed: "No analog muxes: headphone type is selected once with solder links before installation."
- note removed: "REVIEW DRAFT | Labels are electrical connections across all sheets"
- note removed: "TP1-TP4 are direct driver solder pads. There is no jack and no common audio return."
- note removed: "TURBO / planar: bridge each 3-pad selector 2-3; close all four TURBO INPUT links; JP9=2-3."
Changed lines of the file:
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@@
 		(comment 1 "NOT FOR FABRICATION - see DESIGN_NOTES.md")
-	)
-	(text "L-/R- are driven outputs. OPA1688 current does not establish the original 250mW/18ohm target."
-		(exclude_from_sim no)
-		(at 242.062 191.77 0)
-		(effects
-			(font
-				(size 1.27 1.27)
-			)
-			(justify left top)
-		)
-	)
-	(text "REVIEW DRAFT  |  Labels are electrical connections across all sheets"
-		(exclude_from_sim no)
-		(at 245.364 98.424 0)
-		(effects
-			(font
-				(size 1.27 1.27)
-			)
-			(justify left top)
-		)
-	)
-	(text "Eco may omit U5/U8, U4, Q1/Q2 and amplifier support parts entirely. Turbo populates them."
-		(exclude_from_sim no)
-		(at 242.062 181.61 0)
-		(effects
-			(font
-				(size 1.27 1.27)
-			)
-			(justify left top)
-		)
-	)
-	(text "TP1-TP4 are direct driver solder pads. There is no jack and no common audio return."
-		(exclude_from_sim no)
-		(at 242.062 186.69 0)
-		(effects
-			(font
-				(size 1.27 1.27)
-			)
-			(justify left top)
-		)
-	)
-	(text "No analog muxes: headphone type is selected once with solder links before installation."
-		(exclude_from_sim no)
-		(at 242.062 166.37 0)
-		(effects
-			(font
-				(size 1.27 1.27)
-			)
-			(justify left top)
-		)
 	)
 	(text "06 BALANCED OUTPUT"
@@
 			)
 			(justify left top)
-		)
-	)
-	(text "TURBO / planar: bridge each 3-pad selector 2-3; close all four TURBO INPUT links; JP9=2-3."
-		(exclude_from_sim no)
-		(at 242.062 176.53 0)
-		(effects
-			(font
-				(size 1.27 1.27)
-			)
-			(justify left top)
-		)
-	)
-	(text "ECO / HD800: bridge each 3-pad selector 1-2; leave all four TURBO INPUT links open; JP9=1-2."
-		(exclude_from_sim no)
-		(at 242.062 171.45 0)
-		(effects
-			(font
-				(size 1.27 1.27)
-			)
-			(justify left top)
-		)
-	)
-	(text "Configuration links and JP9 must agree before power-up; this design does not hot-switch modes."
-		(exclude_from_sim no)
-		(at 242.062 196.85 0)
-		(effects
-			(font
-				(size 1.27 1.27)
-			)
-			(justify left top)
